File: pcb/SignalGenerator/SignalGenerator.sch (KiCad schematic (older format))
At the start: 29 parts, among them J1 ul.f antenna connector, U1 16 MHz, U2 MIC5205-3.3YM5, U3 AD9837, U4 AD8045

Commit message: Agrego routeo del PCB
Parts:
- U3: footprint Package_SO:MSOP-10_3x3mm_P0.5mm -> generador:LFCSP-WD-10-1EP_3x3mm_P0.5mm_EP1.64x2.38mm
Changed lines of the file:
@@
 F 0 "U3" H 4250 5850 50  0000 L CNN
 F 1 "AD9837" H 4150 5750 50  0000 L CNN
-F 2 "Package_SO:MSOP-10_3x3mm_P0.5mm" H 3950 4700 50  0001 C CNN
+F 2 "generador:LFCSP-WD-10-1EP_3x3mm_P0.5mm_EP1.64x2.38mm" H 3950 4700 50  0001 C CNN
 F 3 "https://www.analog.com/media/en/technical-documentation/data-sheets/ad9833.pdf" H 3900 5600 50  0001 C CNN
 	1    3950 5300

Commit message: Cambios solicitados por el docente
Parts:
- added FID1, FID2: Fiducial, Fiducial:Fiducial_0.5mm_Mask1mm, symbol Mechanical:Fiducial
- LED1: footprint Resistor_SMD:R_0603_1608Metric -> LED_SMD:LED_0603_1608Metric
Other:
- note added: "Clock generator"
- note added: "Fiducials"
- note added: "Power adaptation"
- note added: "Shield header"
- note added: "Signal amplifier"
- note added: "Signal generator"
- moved on the sheet: C1, C13, C2, C3, JP1, JP3, LED1, R1, SJ1, U2

Commit message: Agrego manufacturer, mnf Part Number, Supplier y Supplier PN para los componentes importantes
Parts:
- U2: Manufacturer (none) -> Microchip Technology; Manufacturer Part N. (none) -> MIC5205-3.3YM5-TR; Supplier (none) -> Mouser; Supplier Part N. (none) -> 998-MIC5205-3.3YM5TR
- U3: Manufacturer (none) -> Analog Devices; Manufacturer Part N. (none) -> AD9837ACPZ-RL7; Supplier (none) -> Mouser; Supplier Part N. (none) -> 584-AD9837ACPZ-R7
- U4: Manufacturer (none) -> Analog Devices; Manufacturer Part N. (none) -> AD8045ARDZ; Supplier (none) -> Mouser; Supplier Part N. (none) -> 584-AD8045ARDZ
Changed lines of the file:
@@
 F 2 "generador:LFCSP-WD-10-1EP_3x3mm_P0.5mm_EP1.64x2.38mm" H 3950 4700 50  0001 C CNN
 F 3 "https://www.analog.com/media/en/technical-documentation/data-sheets/ad9833.pdf" H 3900 5600 50  0001 C CNN
+F 4 "Analog Devices" H 3950 5300 50  0001 C CNN "Manufacturer"
+F 5 "AD9837ACPZ-RL7" H 3950 5300 50  0001 C CNN "Manufacturer Part N."
+F 6 "Mouser" H 3950 5300 50  0001 C CNN "Supplier"
+F 7 "584-AD9837ACPZ-R7" H 3950 5300 50  0001 C CNN "Supplier Part N."
 	1    3950 5300
 	1    0    0    -1
@@
 F 2 "Package_TO_SOT_SMD:SOT-23-5" H 2150 3025 50  0001 C CNN
 F 3 "http://ww1.microchip.com/downloads/en/DeviceDoc/20005785A.pdf" H 2150 2700 50  0001 C CNN
+F 4 "Microchip Technology" H 2150 2700 50  0001 C CNN "Manufacturer"
+F 5 "MIC5205-3.3YM5-TR" H 2150 2700 50  0001 C CNN "Manufacturer Part N."
+F 6 "Mouser" H 2150 2700 50  0001 C CNN "Supplier"
+F 7 "998-MIC5205-3.3YM5TR" H 2150 2700 50  0001 C CNN "Supplier Part N."
 	1    2150 2700
 	1    0    0    -1
@@
 F 2 "Package_SO:SOIC-8_3.9x4.9mm_P1.27mm" H 7900 5100 50  0001 L CNN
 F 3 "" H 8150 5450 50  0001 C CNN
+F 4 "Analog Devices" H 8000 5300 50  0001 C CNN "Manufacturer"
+F 5 "AD8045ARDZ" H 8000 5300 50  0001 C CNN "Manufacturer Part N."
+F 6 "Mouser" H 8000 5300 50  0001 C CNN "Supplier"
+F 7 "584-AD8045ARDZ" H 8000 5300 50  0001 C CNN "Supplier Part N."
 	1    8000 5300
 	1    0    0    -1
